File: Balance/ESP_LoRa_Scale_V1.60.brd (EAGLE design)
At the start: 84 x 57.9 mm, 89 parts, among them J1 U.FL, Q1 SI2305CDS, Q2 BSS131, Q3 BSS138, Q4 SI2305CDS, Q5 BSS138, U1 ESP-WROOM-03, U2 NAU7802SOIC, U3 WIRELESS-LORA-RFM95W#SMD, U4 NAU7802SOIC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

Commit message: Add files via upload
Parts:
- added X1: B2B-PH-K-S, con-JST PH:B2B-PH-K-S
- renumbered U5 to U5A, U6 to U5B
Connections:
- net +12V: now also X1.2
- net GND: now also X1.1
Routing:
- net GND: track 449.5 -> 453.3 mm, vias 65 -> 64
- net +12V: track 98.3 -> 99.7 mm
- net VCC: track 195.5 -> 194.5 mm
- net V+: track 163.1 -> 162.6 mm
Other:
- board text added: "+12V"
- board text added: "gnd"
- board text added: "sda scl 3.3 3.3 12 12"
- board text removed: "sda scl 3.3 3.3 +12 +12"
