File: Balance/ESP_LoRa_Scale_V1.60.sch (EAGLE design)
At the start: 89 parts, among them J1 U.FL, Q1 SI2305CDS, Q2 BSS131, Q3 BSS138, Q4 SI2305CDS, Q5 BSS138, U1 ESP-WROOM-03, U2 NAU7802SOIC, U3 WIRELESS-LORA-RFM95W#SMD, U4 NAU7802SOIC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

Commit message: Add files via upload
Parts:
- removed U5: MIC5239 3.3V, micrel:MIC5239-ADJMM
- removed U6: MIC5239S, micrel:MIC5239S
- added U5A: MIC5239 3.3V, micrel:MIC5239-ADJMM
- added U5B: MIC5239S, micrel:MIC5239S
- added X1: B2B-PH-K-S, con-JST PH:B2B-PH-K-S
Connections:
- net +12V: now also U5A.EN, U5A.IN, U5B.IN, X1.2; no longer U5.EN, U5.IN, U6.IN
- net ADJ/FLAG: now also U5A.ADJ; no longer U5.ADJ
- net GND: now also U5A.GND, U5B.GND, X1.1; no longer U5.GND, U6.GND
- net VCC: now also U5A.OUT, U5B.OUT; no longer U5.OUT, U6.OUT
Other:
- note added: "external power (3.6V - 30 V) use U5A or U5B R29 + PWR_ERR LED (with U6 only optional) 20 uA @ 3.6 V ; 22 uA @ 12 V (Iout =0)"
- note removed: "external power (3.6V - 30 V) use U5 or U6 R29 + PWR_ERR LED (with U6 only optional) 20 uA @ 3.6 V ; 22 uA @ 12 V (Iout =0)"
- moved on the sheet: C12, C13, PWR_ERR, R29
